File: auxFilter.kicad_pcb (KiCad board)
At the start: 2 copper layers, 51.6 x 22.8 mm, 27 parts, among them J1 Conn_INPUT, J2 Conn_OUTPUT, U1 4066, U2 AD8668ARZ

Commit message: Added some new images. Changed analog switch part No to one that can handle more than 5v.
Other:
- board text added: "V+"
- board text removed: "5V"
