File: auxFilter.sch (KiCad schematic (older format))
At the start: 27 parts, among them J1 Conn_INPUT, J2 Conn_OUTPUT, U1 4066, U2 AD8668ARZ

Commit message: Added some new images. Changed analog switch part No to one that can handle more than 5v.
Parts:
- U1: digikey 1727-2811-1-ND -> MC14066BDR2GOSCT-ND
Changed lines of the file:
@@
 F 1 "4066" H 4150 1550 50  0000 C CNN
 F 2 "Housings_SOIC:SOIC-14_3.9x8.7mm_Pitch1.27mm" H 4150 1850 50  0001 C CNN
-F 3 "http://www.ti.com/lit/ds/symlink/cd4066b.pdf" H 4150 1850 50  0001 C CNN
-F 4 "1727-2811-1-ND" H 4150 1850 50  0001 C CNN "digikey"
+F 3 "" H 4150 1850 50  0001 C CNN
+F 4 "MC14066BDR2GOSCT-ND" H 4150 1850 50  0001 C CNN "digikey"
 	1    4150 1850
 	1    0    0    -1
@@
 F 1 "4066" H 4150 3200 50  0000 C CNN
 F 2 "Housings_SOIC:SOIC-14_3.9x8.7mm_Pitch1.27mm" H 4150 3500 50  0001 C CNN
-F 3 "http://www.ti.com/lit/ds/symlink/cd4066b.pdf" H 4150 3500 50  0001 C CNN
-F 4 "1727-2811-1-ND" H 4150 3500 50  0001 C CNN "digikey"
+F 3 "" H 4150 3500 50  0001 C CNN
+F 4 "MC14066BDR2GOSCT-ND" H 4150 3500 50  0001 C CNN "digikey"
 	2    4150 3500
 	1    0    0    -1
@@
 F 1 "4066" H 1500 1700 50  0000 L CNN
 F 2 "Housings_SOIC:SOIC-14_3.9x8.7mm_Pitch1.27mm" H 1250 1700 50  0001 C CNN
-F 3 "http://www.ti.com/lit/ds/symlink/cd4066b.pdf" H 1250 1700 50  0001 C CNN
-F 4 "1727-2811-1-ND" H 1250 1700 50  0001 C CNN "digikey"
+F 3 "" H 1250 1700 50  0001 C CNN
+F 4 "MC14066BDR2GOSCT-ND" H 1250 1700 50  0001 C CNN "digikey"
 	5    1250 1700
 	1    0    0    -1
@@
 F 1 "4066" H 4150 4500 50  0000 C CNN
 F 2 "Housings_SOIC:SOIC-14_3.9x8.7mm_Pitch1.27mm" H 4150 4800 50  0001 C CNN
-F 3 "http://www.ti.com/lit/ds/symlink/cd4066b.pdf" H 4150 4800 50  0001 C CNN
-F 4 "1727-2811-1-ND" H 4150 4800 50  0001 C CNN "digikey"
+F 3 "" H 4150 4800 50  0001 C CNN
+F 4 "MC14066BDR2GOSCT-ND" H 4150 4800 50  0001 C CNN "digikey"
 	3    4150 4800
 	1    0    0    -1
@@
 F 1 "4066" H 4150 6150 50  0000 C CNN
 F 2 "Housings_SOIC:SOIC-14_3.9x8.7mm_Pitch1.27mm" H 4150 6450 50  0001 C CNN
-F 3 "http://www.ti.com/lit/ds/symlink/cd4066b.pdf" H 4150 6450 50  0001 C CNN
-F 4 "1727-2811-1-ND" H 4150 6450 50  0001 C CNN "digikey"
+F 3 "" H 4150 6450 50  0001 C CNN
+F 4 "MC14066BDR2GOSCT-ND" H 4150 6450 50  0001 C CNN "digikey"
 	4    4150 6450
 	1    0    0    -1
